File: pcb/ledify.collab/base/ledify.kicad_pcb (KiCad board)
At the start: 2 copper layers, 12 parts, among them J2 USB_C_Receptacle_USB2.0_16P, U1 ESP32-C6_C5364646, U2 USBLC6-2P6, U4 FUSB302BMPX, U5 LM2678T-5.0/NOPB

Commit message: finished stuff
Parts:
- moved L1 41.2 mm to (115.2, 53.0)
Routing:
- net Net-(D1-cathode): track 0.00 -> 93.4 mm, vias 0 -> 16
- net unconnected-(L1-Pad1): track 0.00 -> 21.6 mm
- net (no net): track 0.00 -> 10.7 mm
