File: pcb/ledify.collab/base/ledify.kicad_sch (KiCad schematic)
At the start: 10 parts, among them J2 USB_C_Receptacle_USB2.0_16P, U1 ESP32-C6_C5364646, U2 USBLC6-2P6, U3 AP63203WU, U4 FUSB302BMPX, U6 LM61495QRPHRQ1, U7 TPS56A37RPAR

Commit message: finished stuff
Parts:
- removed U7: TPS56A37RPAR, lcsc:VQFN-HR-10_L3.0-W3.0_TI_RPA, symbol lcsc:TPS56A37RPAR
- added AE1: Antenna_Shield, RF_Antenna:Texas_SWRA117D_2.4GHz_Right, symbol Device:Antenna_Shield
- added C10, C11, C12, C13, C14, C17, C18: 22uF, Capacitor_SMD:C_0805_2012Metric, symbol Device:C
- added C15, C29, C5, C7: 10uF, Capacitor_SMD:C_0603_1608Metric, symbol Device:C
- added C16, C19, C20, C24, C26, C27, C30, C31, C4: 100nF, Capacitor_SMD:C_0402_1005Metric, symbol Device:C
- added C21, C25, C28, C33: 1uF, Capacitor_SMD:C_0402_1005Metric, symbol Device:C
- added C22, C23: 400pF, Capacitor_SMD:C_0402_1005Metric, symbol Device:C
- added C32: 10nF, Capacitor_SMD:C_0402_1005Metric, symbol Device:C
- added C6, C8: 470nF, Capacitor_SMD:C_0402_1005Metric, symbol Device:C
- added C9: 1uF, Capacitor_SMD:C_0603_1608Metric, symbol Device:C
- added L1: ZEMS1770-6R8M, lcsc:IND-SMD_L17.5-W17.5_SLO1770H, symbol lcsc:ZEMS1770-6R8M
- added L2: XRCD43-3R9M, lcsc:IND-SMD_L4.0-W3.2_XRCD43, symbol lcsc:XRCD43-3R9M
- added L3: VHF160808H2N0ST, lcsc:L0603, symbol lcsc:VHF160808H2N0ST
- added Q1: 2N7002K, Package_TO_SOT_SMD:SOT-23, symbol Transistor_FET:2N7002K
- added R1, R2: 100K, Resistor_SMD:R_0402_1005Metric, symbol Device:R
- added R3: 24.9K, Resistor_SMD:R_0402_1005Metric, symbol Device:R
- added R4: 14.3K, Resistor_SMD:R_0402_1005Metric, symbol Device:R
- added R5, R6, R7, R8: 4.7K, Resistor_SMD:R_0402_1005Metric, symbol Device:R
- added SW1: TS-1088-AR02016, lcsc:SW-SMD_L3.9-W3.0-P4.45, symbol lcsc:TS-1088-AR02016
- added U5: W25Q128JVP, Package_SON:WSON-8-1EP_6x5mm_P1.27mm_EP3.4x4.3mm, symbol Memory_Flash:W25Q128JVP
- added X1: XL2EL89COI-111YLC-40M, lcsc:CRYSTAL-SMD_4P-L3.2-W2.5-BL, symbol lcsc:XL2EL89COI-111YLC-40M
- C1: footprint Package_TO_SOT_SMD:SOT-666 -> Capacitor_SMD:C_0603_1608Metric
- C2, C3: footprint Package_TO_SOT_SMD:SOT-666 -> Capacitor_SMD:C_0402_1005Metric
Connections:
- net DM: now also U1.18 (GPIO12)
- net DP: now also U1.19 (GPIO13)
- net GND: now also U3.4 (GND), U6.1 (PGND2), U6.12 (SYNC/MODE), U6.15 (PGND1), U6.8 (AGND), AE1.2 (Shield), C10.2, C11.2, C12.2, C13.2, C14.2, C15.2, C17.2, C18.2, C19.2, C20.2, C21.2, C22.2, C23.2, C24.2, C25.2, C26.2, C27.2, C28.2, C29.2, C30.2, C31.2, C32.2, C33.2, C5.2, C6.2, C7.2, C8.2, C9.2, Q1.2 (S), R3.2, SW1.2, U5.4 (GND), U5.9 (EP), X1.2 (GND), X1.4 (GND)
- net VBUS: now also U3.2 (EN), U3.3 (IN), U6.14 (VIN1), U6.2 (VIN2), C15.1, C5.1, C6.1, C7.1, C8.1
- net at U1.1 (ANT): now also AE1.1 (A)
- net CHIP_EN: now reaches U1.14 (GPIO8)
- net CHIP_EN: now also U1.4 (CHIP_PU), R8.2, SW1.1
- net VDD_A3P: now reaches U1.2 (VDDA3P3)
- net VDD_A3P: now also U1.3 (VDDA3P3), C31.1, L3.1
- net SPICS0: now reaches U1.20 (SPICS0)
- net SPICS0: now also U5.1 (~{CS})
- net SPIQ: now reaches U1.21 (SPIQ)
- net SPIQ: now also U5.2 (DO/IO_{1})
- net SPIWP: now reaches U1.22 (SPIWP)
- net SPIWP: now also U5.3 (~{WP}/IO_{2})
- net +3V3: now reaches U1.23 (VDD_SPI)
- net +3V3: now also U1.28 (VDDPST2), U1.37 (VDDA1), U1.40 (VDDA2), U1.5 (VDDPST1), U3.1 (FB), U4.12 (VCONN), U4.13 (VCONN), U4.3 (VDD), U4.4 (VDD), C17.1, C18.1, C19.1, C20.1, C21.1, C24.1, C25.1, C26.1, C27.1, C28.1, C29.1, C30.1, C32.1, C33.1, L2.2, L3.2, R5.1, R6.1, R7.1, R8.1, U5.8 (VCC)
- net SPIHD: now reaches U1.24 (SPIHD)
- net SPIHD: now also U5.7 (~{HOLD}/~{RESET}/IO_{3})
- net SPICLK: now reaches U1.25 (SPICLK)
- net SPICLK: now also U5.6 (CLK)
- net SPID: now reaches U1.26 (SPID)
- net SPID: now also U5.5 (DI/IO_{0})
- net OSC_IN: now reaches U1.38 (XTAL_N)
- net OSC_IN: now also C23.1, X1.3
- net OSC_OUT: now reaches U1.39 (XTAL_P)
- net OSC_OUT: now also C22.1, X1.1
- net at U6.10 (~{RESET}): now also R1.1
- net at U6.11 (SPSP): now also U6.6 (VCC), U6.9 (RT), C9.1
- net LED_ENABLE: now reaches U6.13 (EN)
- net at U6.16 (SW): now also C4.1, L1.1
- net at U6.3 (RBOOT): now also U6.4 (CBOOT), C4.2
- net LED_VCC: now reaches U6.5 (BIAS)
- net LED_VCC: now also C10.1, C11.1, C12.1, C13.1, C14.1, L1.2, R1.2, R2.1
- net at U6.7 (FB): now also R2.2, R3.1, R4.1
- net at U3.5 (SW): now also C16.2, L2.1
- net at U3.6 (BST): now also C16.1
- net USB_PD_INT: now reaches U4.5 (INT_N)
- net USB_PD_INT: now also R5.2
- net USB_PD_SCL: now reaches U4.6 (SCL)
- net USB_PD_SCL: now also R6.2
- net USB_PD_SDA: now reaches U4.7 (SDA)
- net USB_PD_SDA: now also R7.2
- new net: Q1.3 (D), R4.2
- no-connect marks 2 -> 3
Other:
- moved on the sheet: U1, U3, U6
