File: pcb/ledify.kicad_sch (KiCad schematic)
At the start: 10 parts, among them J2 USB_C_Receptacle_USB2.0_16P, U1 ESP32-C6_C5364646, U2 USBLC6-2P6, U3 AP63203WU, U4 FUSB302BMPX, U6 LM61495QRPHRQ1, U7 TPS56A37RPAR

Commit message: finished stuff
Parts:
- removed U7: TPS56A37RPAR, lcsc:VQFN-HR-10_L3.0-W3.0_TI_RPA, symbol lcsc:TPS56A37RPAR
- added AE1: Antenna_Shield, RF_Antenna:Texas_SWRA117D_2.4GHz_Right, symbol Device:Antenna_Shield
- added C10, C11, C12, C13, C14: 22uF, Capacitor_SMD:C_1210_3225Metric, symbol Device:C
- added C15: 10uF, Capacitor_SMD:C_0805_2012Metric, symbol Device:C
- added C16, C19, C20, C24, C26, C27, C30, C31, C37, C38, C39, C40: 100nF, Capacitor_SMD:C_0402_1005Metric, symbol Device:C
- added C17, C18: 22uF, Capacitor_SMD:C_0805_2012Metric, symbol Device:C
- added C21, C25, C28, C33: 1uF, Capacitor_SMD:C_0402_1005Metric, symbol Device:C
- added C22, C23: 12pF, Capacitor_SMD:C_0402_1005Metric, symbol Device:C
- added C29: 10uF, Capacitor_SMD:C_0603_1608Metric, symbol Device:C
- added C32: 10nF, Capacitor_SMD:C_0402_1005Metric, symbol Device:C
- added C34, C35: 17pF, Capacitor_SMD:C_0402_1005Metric, symbol Device:C
- added C36, C9: 1uF, Capacitor_SMD:C_0603_1608Metric, symbol Device:C
- added C4: 100nF, Capacitor_SMD:C_0402_1005Metric_Pad0.74x0.62mm_HandSolder, symbol Device:C
- added C41: 4pF, Capacitor_SMD:C_0402_1005Metric, symbol Device:C
- added C42: 4.6pF, Capacitor_SMD:C_0402_1005Metric, symbol Device:C
- added C5, C7: 10uF 50V, Capacitor_SMD:C_0805_2012Metric, symbol Device:C
- added C6, C8: 470nF, Capacitor_SMD:C_0603_1608Metric, symbol Device:C
- added H1: MountingHole, MountingHole:MountingHole_2.2mm_M2_Pad_Via, symbol Mechanical:MountingHole
- added J1, J3, J4: Conn_01x01_Pin, Connector_Wire:SolderWirePad_1x01_SMD_3x6mm, symbol Connector:Conn_01x01_Pin
- added L1: ZEMS1770-6R8M, lcsc:IND-SMD_L17.5-W17.5_SLO1770H, symbol lcsc:ZEMS1770-6R8M
- added L2: XRCD43-3R9M, lcsc:IND-SMD_L4.0-W3.2_XRCD43, symbol lcsc:XRCD43-3R9M
- added L3: VHF160808H2N0ST, lcsc:L0603, symbol lcsc:VHF160808H2N0ST
- added L5: TCGL1005B1N8SAT, lcsc:L0402, symbol lcsc:TCGL1005B1N8SAT
- added Q1: 2N7002K, Package_TO_SOT_SMD:SOT-23, symbol Transistor_FET:2N7002K
- added R1, R2: 100K, Resistor_SMD:R_0402_1005Metric, symbol Device:R
- added R3: 24.9K, Resistor_SMD:R_0402_1005Metric, symbol Device:R
- added R4: 14.3K, Resistor_SMD:R_0402_1005Metric, symbol Device:R
- added R5, R6, R7, R8, R9: 4.7K, Resistor_SMD:R_0402_1005Metric, symbol Device:R
- added SW1, SW2: TS-1088-AR02016, lcsc:SW-SMD_L3.9-W3.0-P4.45, symbol lcsc:TS-1088-AR02016
- added U5: W25Q128JVP, Package_SON:WSON-8-1EP_6x5mm_P1.27mm_EP3.4x4.3mm, symbol Memory_Flash:W25Q128JVP
- added U7: BMI323, lcsc:LGA-14_L3.0-W2.5-P0.50-TL_QMI8658A, symbol lcsc:BMI323
- added U8: BMP581, lcsc:LGA-10_L2.0-W2.0-P0.50-TL_BMP581, symbol lcsc:BMP581
- added X1: XL2EL89COI-111YLC-40M, lcsc:CRYSTAL-SMD_4P-L3.2-W2.5-BL, symbol lcsc:XL2EL89COI-111YLC-40M
- added X2: Q13FC1350000400, lcsc:FC-135R_L3.2-W1.5, symbol lcsc:Q13FC1350000400
- C1: value 4.7uF -> 4.7uF 50V; footprint Package_TO_SOT_SMD:SOT-666 -> Capacitor_SMD:C_0603_1608Metric
- C2, C3: footprint Package_TO_SOT_SMD:SOT-666 -> Capacitor_SMD:C_0402_1005Metric
- J2: footprint Package_DFN_QFN:Texas_X2QFN-12_1.6x1.6mm_P0.4mm -> Connector_USB:USB_C_Receptacle_HCTL_HC-TYPE-C-16P-01A
Connections:
- net DM is gone; now on net DN: U2.6 (I/O1)
- net DP: now also U1.19 (GPIO13)
- net GND: now also U3.4 (GND), U6.1 (PGND2), U6.12 (SYNC/MODE), U6.15 (PGND1), U6.8 (AGND), AE1.2 (Shield), C10.2, C11.2, C12.2, C13.2, C14.2, C15.2, C17.2, C18.2, C19.2, C20.2, C21.2, C22.2, C23.2, C24.2, C25.2, C26.2, C27.2, C28.2, C29.2, C30.2, C31.2, C32.2, C33.2, C34.2, C35.2, C36.2, C37.2, C38.2, C39.2, C40.2, C41.2, C42.2, C5.2, C6.2, C7.2, C8.2, C9.2, J4.1 (Pin_1), Q1.2 (S), R3.2, R9.2, SW1.2, SW2.2, U5.4 (GND), U5.9 (EP), U7.6 (GNDIO), U7.7 (GND), U8.3 (VSS), U8.8 (VSS), U8.9 (VSS), X1.2 (GND), X1.4 (GND)
- net VBUS: now also U3.2 (EN), U3.3 (IN), U6.14 (VIN1), U6.2 (VIN2), C15.1, C5.1, C6.1, C7.1, C8.1
- net at U1.1 (ANT): now also C42.1, L5.2
- net CHIP_BOOT: now reaches U1.14 (GPIO8)
- net CHIP_BOOT: now also SW2.1
- net DN: now reaches U1.18 (GPIO12)
- net VDD_A3P: now reaches U1.2 (VDDA3P3)
- net VDD_A3P: now also U1.3 (VDDA3P3), C31.1, L3.1
- net SPICS0: now reaches U1.20 (SPICS0)
- net SPICS0: now also U5.1 (~{CS})
- net SPIQ: now reaches U1.21 (SPIQ)
- net SPIQ: now also U5.2 (DO/IO_{1})
- net SPIWP: now reaches U1.22 (SPIWP)
- net SPIWP: now also U5.3 (~{WP}/IO_{2})
- net +3V3: now reaches U1.23 (VDD_SPI)
- net +3V3: now also U1.28 (VDDPST2), U1.37 (VDDA1), U1.40 (VDDA2), U1.5 (VDDPST1), U3.1 (FB), U4.12 (VCONN), U4.13 (VCONN), U4.3 (VDD), U4.4 (VDD), C17.1, C18.1, C19.1, C20.1, C21.1, C24.1, C25.1, C26.1, C27.1, C28.1, C29.1, C30.1, C32.1, C33.1, C37.1, C38.1, C39.1, C40.1, L2.2, L3.2, R5.1, R6.1, R7.1, R8.1, U5.8 (VCC), U7.5 (VDDIO), U7.8 (VDD), U8.1 (VDDIO), U8.10 (VDD)
- net SPIHD: now reaches U1.24 (SPIHD)
- net SPIHD: now also U5.7 (~{HOLD}/~{RESET}/IO_{3})
- net SPICLK: now reaches U1.25 (SPICLK)
- net SPICLK: now also U5.6 (CLK)
- net SPID: now reaches U1.26 (SPID)
- net SPID: now also U5.5 (DI/IO_{0})
- net LED_CON: now reaches U1.27 (GPIO15)
- net LED_CON: now also J3.1 (Pin_1)
- net SPI_MISO: now reaches U1.31 (SDIO_CMD)
- net SPI_MISO: now also U7.1 (SDO), U8.5 (SDO)
- net SPI_MOSI: now reaches U1.32 (SDIO_CLK)
- net SPI_MOSI: now also U7.14 (SDX), U8.4 (SDI)
- net SPI_SCK: now reaches U1.33 (SDIO_DATA0)
- net SPI_SCK: now also U7.13 (SCX), U8.2 (SCK)
- net CS_IMU: now reaches U1.34 (SDIO_DATA1)
- net CS_IMU: now also U7.12 (CSB)
- net CS_BARO: now reaches U1.35 (SDIO_DATA2)
- net CS_BARO: now also U8.6 (CSB)
- net OSC_IN: now reaches U1.38 (XTAL_N)
- net OSC_IN: now also C23.1, X1.3
- net OSC_OUT: now reaches U1.39 (XTAL_P)
- net OSC_OUT: now also C22.1, X1.1
- net CHIP_EN: now reaches U1.4 (CHIP_PU)
- net CHIP_EN: now also C36.1, R8.2, SW1.1
- net OSC_32_OUT: now reaches U1.6 (XTAL_32K_P)
- net OSC_32_OUT: now also C34.1, X2.1
- net OSC_32_IN: now reaches U1.7 (XTAL_32K_N)
- net OSC_32_IN: now also C35.1, X2.2
- net LED_SW_V: now reaches U1.8 (GPIO2)
- net LED_SW_V: now also Q1.1 (G), R9.1
- net LED_ENABLE: now reaches U1.9 (GPIO3)
- net LED_ENABLE: now also U6.13 (EN)
- net at U6.10 (~{RESET}): now also R1.1
- net at U6.11 (SPSP): now also U6.6 (VCC), U6.9 (RT), C9.1
- net at U6.16 (SW): now also C4.1, L1.1
- net at U6.3 (RBOOT): now also U6.4 (CBOOT), C4.2
- net LED_VCC: now reaches U6.5 (BIAS)
- net LED_VCC: now also C10.1, C11.1, C12.1, C13.1, C14.1, J1.1 (Pin_1), L1.2, R1.2, R2.1
- net at U6.7 (FB): now also R2.2, R3.1, R4.1
- net at U3.5 (SW): now also C16.2, L2.1
- net at U3.6 (BST): now also C16.1
- net USB_PD_INT: now reaches U4.5 (INT_N)
- net USB_PD_INT: now also R5.2
- net USB_PD_SCL: now reaches U4.6 (SCL)
- net USB_PD_SCL: now also R6.2
- net USB_PD_SDA: now reaches U4.7 (SDA)
- net USB_PD_SDA: now also R7.2
- new net: Q1.3 (D), R4.2
- new net: AE1.1 (A), C41.1, L5.1
- no-connect marks 2 -> 20
Other:
- note added: "3V3 Buck"
- note added: "Barometer"
- note added: "Buttons"
- note added: "Crystals"
- note added: "Decoupling Capacitors"
- note added: "ESP32"
- note added: "Flash"
- note added: "IMU"
- note added: "LED Buck"
- note added: "USB-C"
- note added: "USB-C PD"
- moved on the sheet: C1, C2, C3, J2, U1, U2, U3, U4, U6

Commit message: aaa
Parts:
- C1: value 4.7uF 50V -> 4.7uF 25V; LCSC (none) -> C69335
- C10, C11, C12, C13, C14: value 22uF -> 22uF 25V; LCSC (none) -> C309062
- C2, C3: LCSC (none) -> C76971
- C41: LCSC (none) -> C541337
- C42: LCSC (none) -> C1855288
- J2: LCSC (none) -> C2894897
- R4: LCSC (none) -> C25855
- U3: LCSC (none) -> C780769
- U5: LCSC (none) -> C2441427
Changed lines of the file:
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@@
 			)
 		)
+		(property "LCSC" "C2441427"
+			(at 262.89 81.28 0)
+			(hide yes)
+			(show_name no)
+			(do_not_autoplace no)
+			(effects
+				(font
+					(size 1.27 1.27)
+				)
+			)
+		)
 		(pin "5"
 		)
@@
 			)
 		)
+		(property "LCSC" "C25855"
+			(at 358.14 194.31 0)
+			(hide yes)
+			(show_name no)
+			(do_not_autoplace no)
+			(effects
+				(font
+					(size 1.27 1.27)
+				)
+			)
+		)
 		(pin "2"
 		)
@@
 			)
 		)
+		(property "LCSC" "C76971"
+			(at 115.57 132.08 0)
+			(hide yes)
+			(show_name no)
+			(do_not_autoplace no)
+			(effects
+				(font
+					(size 1.27 1.27)
+				)
+			)
+		)
 		(pin "2"
 		)
@@
 			)
 		)
+		(property "LCSC" "C541337"
+			(at 311.15 83.82 0)
+			(hide yes)
+			(show_name no)
+			(do_not_autoplace no)
+			(effects
+				(font
+					(size 1.27 1.27)
+				)
+			)
+		)
 		(pin "2"
 		)
@@
 		(dnp no)
 		(property "Reference" "C13"
-			(at 336.804 178.054 0)
+			(at 336.804 177.546 0)
 			(show_name no)
 			(do_not_autoplace no)
@@
 			)
 		)
-		(property "Value" "22uF"
-			(at 336.804 180.086 0)
+		(property "Value" "22uF\n25V"
+			(at 336.804 180.34 0)
 			(show_name no)
 			(do_not_autoplace no)
@@
 			)
 		)
+		(property "LCSC" "C309062"
+			(at 334.01 179.07 0)
+			(hide yes)
+			(show_name no)
+			(do_not_autoplace no)
+			(effects
+				(font
+					(size 1.27 1.27)
+				)
+			)
+		)
 		(pin "2"
 		)
@@
 			)
 		)
+		(property "LCSC" "C780769"
+			(at 212.09 265.43 0)
+			(hide yes)
+			(show_name no)
+			(do_not_autoplace no)
+			(effects
+				(font
+					(size 1.27 1.27)
+				)
+			)
+		)
 		(pin "2"
 		)
@@
 			)
 		)
+		(property "LCSC" "C2894897"
+			(at 45.72 44.45 0)
+			(hide yes)
+			(show_name no)
+			(do_not_autoplace no)
+			(effects
+				(font
+					(size 1.27 1.27)
+				)
+			)
+		)
 		(pin "B6"
 		)
@@
 			)
 		)
-		(property "Value" "4.7uF\n50V"
+		(property "Value" "4.7uF\n25V"
 			(at 73.914 35.306 0)
 			(show_name no)
@@
 			)
 		)
+		(property "LCSC" "C69335"
+			(at 71.12 33.02 0)
+			(hide yes)
+			(show_name no)
+			(do_not_autoplace no)
+			(effects
+				(font
+					(size 1.27 1.27)
+				)
+			)
+		)
 		(pin "2"
 		)
@@
 			)
 		)
+		(property "LCSC" "C1855288"
+			(at 326.39 83.82 0)
+			(hide yes)
+			(show_name no)
+			(do_not_autoplace no)
+			(effects
+				(font
+					(size 1.27 1.27)
+				)
+			)
+		)
 		(pin "2"
 		)
@@
 		(dnp no)
 		(property "Reference" "C11"
-			(at 315.214 178.054 0)
+			(at 315.214 177.546 0)
 			(show_name no)
 			(do_not_autoplace no)
@@
 			)
 		)
-		(property "Value" "22uF"
-			(at 315.214 180.086 0)
+		(property "Value" "22uF\n25V"
+			(at 315.214 180.34 0)
 			(show_name no)
 			(do_not_autoplace no)
@@
 			)
 		)
+		(property "LCSC" "C309062"
+			(at 312.42 179.07 0)
+			(hide yes)
+			(show_name no)
+			(do_not_autoplace no)
+			(effects
+				(font
+					(size 1.27 1.27)
+				)
+			)
+		)
 		(pin "2"
 		)
@@
 			)
 		)
+		(property "LCSC" "C76971"
+			(at 110.49 132.08 0)
+			(hide yes)
+			(show_name no)
+			(do_not_autoplace no)
+			(effects
+				(font
+					(size 1.27 1.27)
+				)
+			)
+		)
 		(pin "2"
 		)
@@
 		(dnp no)
 		(property "Reference" "C12"
-			(at 326.644 178.054 0)
+			(at 326.644 177.546 0)
 			(show_name no)
 			(do_not_autoplace no)
@@
 			)
 		)
-		(property "Value" "22uF"
-			(at 326.644 180.086 0)
+		(property "Value" "22uF\n25V"
+			(at 326.644 180.34 0)
 			(show_name no)
 			(do_not_autoplace no)
@@
 			)
 		)
+		(property "LCSC" "C309062"
+			(at 323.85 179.07 0)
+			(hide yes)
+			(show_name no)
+			(do_not_autoplace no)
+			(effects
+				(font
+					(size 1.27 1.27)
+				)
+			)
+		)
 		(pin "2"
 		)
@@
 		(dnp no)
 		(property "Reference" "C10"
-			(at 305.054 178.054 0)
+			(at 305.054 177.546 0)
 			(show_name no)
 			(do_not_autoplace no)
@@
 			)
 		)
-		(property "Value" "22uF"
-			(at 305.054 180.086 0)
+		(property "Value" "22uF\n25V"
+			(at 305.054 180.34 0)
 			(show_name no)
 			(do_not_autoplace no)
@@
 			)
 		)
+		(property "LCSC" "C309062"
+			(at 302.26 179.07 0)
+			(hide yes)
+			(show_name no)
+			(do_not_autoplace no)
+			(effects
+				(font
+					(size 1.27 1.27)
+				)
+			)
+		)
 		(pin "2"
 		)
@@
 		(dnp no)
 		(property "Reference" "C14"
-			(at 346.964 178.054 0)
+			(at 346.964 177.546 0)
 			(show_name no)
 			(do_not_autoplace no)
@@
 			)
 		)
-		(property "Value" "22uF"
-			(at 346.964 180.086 0)
+		(property "Value" "22uF\n25V"
+			(at 346.964 180.34 0)
 			(show_name no)
 			(do_not_autoplace no)
@@
 			(at 344.17 179.07 0)
 			(hide yes)
+			(show_name no)
+			(do_not_autoplace no)
+			(effects
+				(font
+					(size 1.27 1.27)
+				)
+			)
+		)
+		(property "LCSC" "C309062"
+			(at 344.17 179.07 0)
+			(hide yes)

Commit message: blender render
Other:
- note added: "Le"
- note added: "di"
- note added: "fy"
- moved on the sheet: C22, C23, C34, C35, R8, SW1, SW2, X1, X2

Commit message: fixes and done
Parts:
- added R10, R11: 4.7K, Resistor_SMD:R_0402_1005Metric, symbol Device:R
- C1: value 4.7uF 25V -> 4.7uF 35V; LCSC C69335 -> C307467
- C15: value 10uF -> 10uF 50V; LCSC (none) -> C440198
- C2, C3: value 400pF -> 470pF
- C22, C23: value 12pF -> 18pF; LCSC (none) -> C1549
- C34, C35: value 17pF -> 18pF; LCSC (none) -> C1549
- C36: footprint Capacitor_SMD:C_0603_1608Metric -> Capacitor_SMD:C_0402_1005Metric
- C5, C7: LCSC (none) -> C440198
- C6: LCSC (none) -> C42371693
- C8: value 470nF -> 470nF 50V; LCSC (none) -> C42371693
Connections:
- net +3V3: now also U2.5 (VBUS), R10.1
- net CHIP_BOOT: now also U1.15 (GPIO9); no longer U1.14 (GPIO8)
- net GND: now also R11.2
- net LED_ENABLE: now also R11.1
- net USB_PD_INT: now also U1.29 (U0TXD)
- net USB_PD_SCL: now also U1.17 (GPIO11)
- net USB_PD_SDA: now also U1.16 (GPIO10)
- net VBUS: no longer U2.5 (VBUS)
- new net: R10.2, U1.14 (GPIO8)
- no-connect marks 20 -> 16
Other:
- moved on the sheet: AE1, C36, C41, C42, L5, U1

Commit message: add light sensor and i2s mic, fix ground return paths, update journal
Parts:
- added C43, C44: 100nF, Capacitor_SMD:C_0402_1005Metric, symbol Device:C
- added U10: OPT4001DNPRQ1, lcsc:USON-6_L2.0-W2.0-P0.65-BL-EP, symbol lcsc:OPT4001DNPRQ1
- added U11: ICS-43434_C5656610, lcsc:MIC-SMD_6P-L3.5-W2.7-P0.90-BL, symbol lcsc:ICS-43434_C5656610
- C6: value 470nF -> 470nF 50V; LCSC C42371693 -> C77572
- C8: LCSC C42371693 -> C77572
- U4: LCSC (none) -> C132291
Connections:
- net +3V3: now also C43.1, C44.1, U10.1 (VDD), U11.5 (VDD)
- net CS_BARO: now also U1.13 (MTDO); no longer U1.35 (SDIO_DATA2)
- net GND: now also C43.2, C44.2, U10.2 (ADDR), U10.3 (GND), U10.7 (EP), U11.2 (LR), U11.3 (GND)
- net LED_CON: now also U1.11 (MTDI); no longer U1.27 (GPIO15)
- net MIC_OUT: now reaches U1.12 (MTCK)
- net MIC_OUT: now also U11.6 (SD)
- net MIC_SCK: now reaches U1.36 (SDIO_DATA3)
- net MIC_SCK: now also U11.4 (SCK)
- net USB_PD_SCL renamed I2C_SCL
- net I2C_SCL: now also U10.4 (SCL)
- net USB_PD_SDA renamed I2C_SDA
- net I2C_SDA: now also U10.6 (SDA)
- new net MIC_CS: U1.35 (SDIO_DATA2), U11.1 (WS)
- no-connect marks 16 -> 14
Other:
- note added: "Light Sensor"
- note added: "Microphone"
- moved on the sheet: C37, C38, C39, C40, R8, SW1, SW2, U7, U8
